File: Day_05_Linux_SBC/Day_05_Linux_SBC.kicad_pcb (KiCad board)
At the start: 8 copper layers, 26 x 30 mm, 13 parts, among them J1 USB_C_Plug_USB2.0, J2 Conn_ARM_SWD_TagConnect_TC203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, J3 USB_C_Receptacle_USB2.0_14P, J4 Conn_01x04_MountingPin, J5 Micro_SD_Card_Det2, U1 D3V3XA4B10LP, U2 STM32H503KBUx, U3 RV1106G2, U4 CH334P

Commit message: updates
Parts:
- removed U4: CH334P, Package_DFN_QFN:QFN-16-1EP_3x3mm_P0.5mm_EP1.75x1.75mm
- added AE1: Antenna_Chip, RF_Antenna:Johanson_2450AT18x100_2400-2500Mhz, B.Cu at (160.2, 105.0)
- added U10: TS3USB30ERSWR, Package_DFN_QFN:UQFN-10_1.4x1.8mm_P0.4mm, F.Cu at (152.0, 113.8)
- added U5: ESP32-C6FH4, Package_DFN_QFN:QFN-32-1EP_5x5mm_P0.5mm_EP3.6x3.6mm, B.Cu at (152.8, 105.0)
- added U6: RV1106G2, Framework_Shilling_Library:QFN-128_L12.3-W12.3-P0.35-TL-EP7.0-1, F.Cu at (148.5, 105.0)
- added U7: STEMMA-QT, amemb-Conenctor_JST:JST_SH_SM04B-SRSS-TB_1x04-1MP_P1.00mm_Horizontal, F.Cu at (157.2, 116.5)
- added U8: EA3058QD, Package_DFN_QFN:VQFN-24-1EP_4x4mm_P0.5mm_EP2.5x2.5mm_ThermalVias, F.Cu at (141.0, 94.5)
- added U9: MP2722, amemb-Package_DFN_QFN:QFN-22_MP2722_2.5x3.5mm_P0.4mm, F.Cu at (138.2, 108.5)
- J4: value Conn_01x04_MountingPin -> JST SH SM03B; footprint Connector_JST:JST_SH_SM04B-SRSS-TB_1x04-1MP_P1.00mm_Horizontal -> Connector_JST:JST_SH_SM03B-SRSS-TB_1x03-1MP_P1.00mm_Horizontal; moved to B.Cu
- U3: value RV1106G2 -> CH334P; footprint Framework_Shilling_Library:QFN-128_L12.3-W12.3-P0.35-TL-EP7.0-1 -> Package_DFN_QFN:QFN-16-1EP_3x3mm_P0.5mm_EP1.75x1.75mm
- moved LOGO1 37.6 mm to (171.2, 83.4)
- moved H2 34.4 mm to (142.8, 79.6)
- moved H1 34.4 mm to (120.2, 79.6)
- moved J4 24.9 mm to (139.0, 97.5), turned to 90 degrees
- moved U3 14.1 mm to (157.0, 93.5)
- moved J5 7.35 mm to (142.0, 108.0), turned to 90 degrees
Connections:
- net /SWCLK renamed /STM32H5/SWCLK
- net /SWDIO renamed /STM32H5/SWDIO
- net /~{RESET} renamed /STM32H5/~{RESET}
- J3 pad A5: unconnected-(J3-CC1-PadA5) -> /PMIC.CC1
- J3 pad A6: unconnected-(J3-D+-PadA6) -> /MPU_OUT.D+
- J3 pad A7: unconnected-(J3-D--PadA7) -> /MPU_OUT.D-
- J3 pad B5: unconnected-(J3-CC2-PadB5) -> /PMIC.CC2
- J3 pad B6: unconnected-(J3-D+-PadB6) -> /MPU_OUT.D+
- J3 pad B7: unconnected-(J3-D--PadB7) -> /MPU_OUT.D-
- J4 pad 1: unconnected-(J4-Pin_1-Pad1) -> Net-(J4-Pin_1)
- J4 pad 2: unconnected-(J4-Pin_2-Pad2) -> /Power Supply/NTC
- J4 pad 3: unconnected-(J4-Pin_3-Pad3) -> GND
- J4 pad MP: unconnected-(J4-MountPin-PadMP) -> GND
- U2 pad 14: unconnected-(U2-PB0-Pad14) -> /STM32H5/DEBUG.TX
- U2 pad 15: unconnected-(U2-PB1-Pad15) -> /STM32H5/DEBUG.RX
- U2 pad 21: unconnected-(U2-PA11-Pad21) -> /STM32H5/DEBUG.D-
- U2 pad 22: unconnected-(U2-PA12-Pad22) -> /STM32H5/DEBUG.D+
- U3 pad 10: unconnected-(U3A-DVDD_1-Pad10) -> Net-(U10-D2+)
- U3 pad 11: unconnected-(U3B-SDMMC0_DET-Pad11) -> /D-
- U3 pad 12: unconnected-(U3B-SDMMC0_D1-Pad12) -> /D+
- U3 pad 17: unconnected-(U3B-SDMMC0_D3-Pad17) -> GND
- U3 pad 5: unconnected-(U3D-VI_CIF_D11-Pad5) -> /ESP32.D-
- U3 pad 6: unconnected-(U3D-VI_CIF_D13-Pad6) -> /ESP32.D+
- U3 pad 7: unconnected-(U3D-VI_CIF_D12-Pad7) -> /DEBUG.D-
- U3 pad 8: unconnected-(U3D-VI_CIF_D14-Pad8) -> /DEBUG.D+
- U3 pad 9: unconnected-(U3D-VI_CIF_D15-Pad9) -> Net-(U10-D2-)
Other:
- outline, holes or cut-outs redrawn
- board text removed: "PMIC"

Commit message: updates
Parts:
- added C1: 10uF, amemb-Capacitor_SMD:amemb-C_0402_1005Metric_L, F.Cu at (153.4, 92.0)
- added C10: 220pF, amemb-Capacitor_SMD:amemb-C_0201_0603Metric_L, F.Cu at (145.3, 98.8)
- added C11: 22uF, amemb-Capacitor_SMD:amemb-C_0402_1005Metric_L, F.Cu at (140.7, 93.0)
- added C12: 22uF, amemb-Capacitor_SMD:amemb-C_0402_1005Metric_L, F.Cu at (145.2, 98.2)
- added C13: 22uF, amemb-Capacitor_SMD:amemb-C_0402_1005Metric_L, F.Cu at (142.3, 99.8)
- added C14: 22uF, amemb-Capacitor_SMD:amemb-C_0402_1005Metric_L, F.Cu at (138.8, 94.9)
- added C15: 10uF, amemb-Capacitor_SMD:amemb-C_0402_1005Metric_L, F.Cu at (139.3, 99.3)
- added C16: 10uF, amemb-Capacitor_SMD:amemb-C_0402_1005Metric_L, F.Cu at (143.4, 93.7)
- added C17: 10uF, amemb-Capacitor_SMD:amemb-C_0402_1005Metric_L, F.Cu at (144.4, 94.8)
- added C18: 10uF, amemb-Capacitor_SMD:amemb-C_0402_1005Metric_L, F.Cu at (138.5, 98.4)
- added C19: 10uF, amemb-Capacitor_SMD:amemb-C_0402_1005Metric_L, F.Cu at (143.6, 98.5)
- added C2: 10uF, amemb-Capacitor_SMD:amemb-C_0402_1005Metric_L, F.Cu at (160.4, 96.1)
- added C20: 22nF, amemb-Capacitor_SMD:amemb-C_0201_0603Metric_L, F.Cu at (136.8, 104.0)
- added C21: 1uF, amemb-Capacitor_SMD:amemb-C_0201_0603Metric_L, F.Cu at (139.8, 102.9)
- added C22: 22uF, amemb-Capacitor_SMD:amemb-C_0402_1005Metric_L, F.Cu at (136.9, 101.8)
- added C23: 10uF, amemb-Capacitor_SMD:amemb-C_0402_1005Metric_L, F.Cu at (139.2, 102.7)
- added C24: 4.7uF, amemb-Capacitor_SMD:amemb-C_0402_1005Metric_L, F.Cu at (141.7, 105.6)
- added C25: 1uF, amemb-Capacitor_SMD:amemb-C_0201_0603Metric_L, F.Cu at (142.3, 112.4)
- added C26: 10uF, amemb-Capacitor_SMD:amemb-C_0402_1005Metric_L, B.Cu at (153.6, 115.0)
- added C27: 1uF, amemb-Capacitor_SMD:amemb-C_0201_0603Metric_L, B.Cu at (152.9, 114.8)
- added C28: 1uF, amemb-Capacitor_SMD:amemb-C_0201_0603Metric_L, B.Cu at (152.1, 114.8)
- added C29: 1uF, amemb-Capacitor_SMD:amemb-C_0201_0603Metric_L, B.Cu at (156.0, 112.9)
- added C3: 1uF, amemb-Capacitor_SMD:amemb-C_0201_0603Metric_L, F.Cu at (153.5, 94.7)
- added C30: 1uF, amemb-Capacitor_SMD:amemb-C_0201_0603Metric_L, B.Cu at (151.6, 114.8)
- added C31: 1uF, amemb-Capacitor_SMD:amemb-C_0201_0603Metric_L, B.Cu at (152.1, 107.5)
- added C32: 1uF, amemb-Capacitor_SMD:amemb-C_0201_0603Metric_L, B.Cu at (156.0, 111.3)
- added C33: 1uF, amemb-Capacitor_SMD:amemb-C_0201_0603Metric_L, B.Cu at (156.5, 110.8)
- added C34: 1.2pF, amemb-Capacitor_SMD:amemb-C_01005_0402Metric_L, B.Cu at (155.1, 114.3)
- added C35: 1.2pF, amemb-Capacitor_SMD:amemb-C_01005_0402Metric_L, B.Cu at (156.1, 115.3)
- added C36: 1.2pF, amemb-Capacitor_SMD:amemb-C_01005_0402Metric_L, B.Cu at (158.6, 115.9)
- added C37: 1.2pF, amemb-Capacitor_SMD:amemb-C_01005_0402Metric_L, B.Cu at (157.1, 115.9)
- added C38: 10uF, amemb-Capacitor_SMD:amemb-C_0402_1005Metric_L, B.Cu at (158.4, 102.4)
- added C39: 1uF, amemb-Capacitor_SMD:amemb-C_0201_0603Metric_L, B.Cu at (158.2, 99.5)
- added C4: 10uF, amemb-Capacitor_SMD:amemb-C_0402_1005Metric_L, F.Cu at (159.8, 97.3)
- added C40: 1uF, amemb-Capacitor_SMD:amemb-C_0201_0603Metric_L, B.Cu at (156.8, 99.5)
- added C41: 1uF, amemb-Capacitor_SMD:amemb-C_0201_0603Metric_L, B.Cu at (158.5, 103.6)
- added C42: 1uF, amemb-Capacitor_SMD:amemb-C_0201_0603Metric_L, F.Cu at (160.6, 104.2)
- added C43: 1uF, amemb-Capacitor_SMD:amemb-C_0201_0603Metric_L, F.Cu at (160.8, 102.7)
- added C44: 10uF, amemb-Capacitor_SMD:amemb-C_0402_1005Metric_L, B.Cu at (158.4, 104.3)
- added C45: 10uF, amemb-Capacitor_SMD:amemb-C_0402_1005Metric_L, F.Cu at (160.6, 101.6)
- added C46: 1uF, amemb-Capacitor_SMD:amemb-C_0201_0603Metric_L, B.Cu at (149.4, 106.2)
- added C47: 1uF, amemb-Capacitor_SMD:amemb-C_0201_0603Metric_L, B.Cu at (158.5, 101.7)
- added C48: 1uF, amemb-Capacitor_SMD:amemb-C_0201_0603Metric_L, B.Cu at (153.0, 99.5)
- added C49: 10uF, amemb-Capacitor_SMD:amemb-C_0402_1005Metric_L, B.Cu at (149.6, 105.5)
- added C5: 220pF, amemb-Capacitor_SMD:amemb-C_0201_0603Metric_L, F.Cu at (140.2, 92.5)
- added C50: 1uF, amemb-Capacitor_SMD:amemb-C_0201_0603Metric_L, F.Cu at (146.2, 101.2)
- added C51: 1uF, amemb-Capacitor_SMD:amemb-C_0201_0603Metric_L, F.Cu at (151.2, 111.6)
- added C52: 1uF, amemb-Capacitor_SMD:amemb-C_0201_0603Metric_L, F.Cu at (146.2, 105.5)
- added C53: 1uF, amemb-Capacitor_SMD:amemb-C_0201_0603Metric_L, F.Cu at (156.9, 97.7)
- added C54: 1uF, amemb-Capacitor_SMD:amemb-C_0201_0603Metric_L, F.Cu at (148.1, 111.6)
- added C55: 10uF, amemb-Capacitor_SMD:amemb-C_0402_1005Metric_L, F.Cu at (158.6, 111.8)
- added C56: 1uF, amemb-Capacitor_SMD:amemb-C_0201_0603Metric_L, F.Cu at (154.4, 111.6)
- added C57: 10uF, amemb-Capacitor_SMD:amemb-C_0402_1005Metric_L, F.Cu at (160.6, 99.7)
- added C58: 1uF, amemb-Capacitor_SMD:amemb-C_0201_0603Metric_L, F.Cu at (160.8, 103.2)
- added C59: 1uF, amemb-Capacitor_SMD:amemb-C_0201_0603Metric_L, F.Cu at (150.9, 97.4)
- added C6: 220pF, amemb-Capacitor_SMD:amemb-C_0201_0603Metric_L, F.Cu at (143.9, 100.4)
- added C60: 1uF, amemb-Capacitor_SMD:amemb-C_0201_0603Metric_L, F.Cu at (160.6, 106.4)
- added C61: 1uF, amemb-Capacitor_SMD:amemb-C_0201_0603Metric_L, F.Cu at (152.3, 111.6)
- added C62: 1uF, amemb-Capacitor_SMD:amemb-C_0201_0603Metric_L, F.Cu at (153.3, 97.4)
- added C63: 1uF, amemb-Capacitor_SMD:amemb-C_0201_0603Metric_L, F.Cu at (146.2, 102.9)
- added C64: 10uF, amemb-Capacitor_SMD:amemb-C_0402_1005Metric_L, B.Cu at (151.0, 98.5)
- added C65: 10uF, amemb-Capacitor_SMD:amemb-C_0402_1005Metric_L, B.Cu at (151.0, 100.0)
- added C66: 10uF, amemb-Capacitor_SMD:amemb-C_0402_1005Metric_L, B.Cu at (149.8, 101.2)
- added C7: 220pF, amemb-Capacitor_SMD:amemb-C_0201_0603Metric_L, F.Cu at (138.1, 93.2)
- added C8: 47nF, amemb-Capacitor_SMD:amemb-C_0201_0603Metric_L, F.Cu at (137.8, 99.6)
- added C9: 100nF, amemb-Capacitor_SMD:amemb-C_0201_0603Metric_L, F.Cu at (137.4, 99.2)
- added L1: 1.5uH, amemb-Inductor_SMD:amemb-L_0806_2016Metric_L, F.Cu at (142.6, 92.2)
- added L2: 1.5uH, amemb-Inductor_SMD:amemb-L_0806_2016Metric_L, F.Cu at (140.3, 100.7)
- added L3: 1.5uH, amemb-Inductor_SMD:amemb-L_0806_2016Metric_L, F.Cu at (137.1, 96.6)
- added L4: 1.5uH, amemb-Inductor_SMD:amemb-L_0806_2016Metric_L, F.Cu at (145.6, 96.5)
- added L5: 1uH, amemb-Inductor_SMD:amemb-L_0805_2012Metric_L, F.Cu at (137.5, 102.8)
- added L6: 2.4nH, amemb-Inductor_SMD:amemb-L_0201_0603Metric_L, B.Cu at (155.5, 114.9)
- added L7: 0R, amemb-Resistor_SMD:amemb-R_0201_0603Metric_L, B.Cu at (157.9, 116.1)
- added R1: 5.1kR, amemb-Resistor_SMD:amemb-R_0201_0603Metric_L, F.Cu at (146.8, 94.6)
- added R10: 100kR, amemb-Resistor_SMD:amemb-R_0201_0603Metric_L, F.Cu at (137.1, 98.9)
- added R11: 200kR, amemb-Resistor_SMD:amemb-R_0201_0603Metric_L, F.Cu at (145.3, 99.3)
- added R12: 100kR, amemb-Resistor_SMD:amemb-R_0201_0603Metric_L, F.Cu at (144.5, 99.1)
- added R13: 510kR, amemb-Resistor_SMD:amemb-R_0201_0603Metric_L, F.Cu at (136.6, 105.8)
- added R14: 240R, amemb-Resistor_SMD:amemb-R_0201_0603Metric_L, F.Cu at (160.8, 103.8)
- added R15: 100kR, amemb-Resistor_SMD:amemb-R_0201_0603Metric_L, B.Cu at (152.6, 115.9)
- added R16: 100kR, amemb-Resistor_SMD:amemb-R_0201_0603Metric_L, B.Cu at (149.0, 109.7)
- added R2: 10kR, amemb-Resistor_SMD:amemb-R_0201_0603Metric_L, F.Cu at (155.9, 90.8)
- added R3: 510kR, amemb-Resistor_SMD:amemb-R_0201_0603Metric_L, F.Cu at (139.9, 92.2)
- added R4: 100kR, amemb-Resistor_SMD:amemb-R_0201_0603Metric_L, F.Cu at (139.8, 93.5)
- added R5: 100kR, amemb-Resistor_SMD:amemb-R_0201_0603Metric_L, F.Cu at (143.6, 100.1)
- added R6: 80.6kR, amemb-Resistor_SMD:amemb-R_0201_0603Metric_L, F.Cu at (143.2, 99.7)
- added R7: 100kR, amemb-Resistor_SMD:amemb-R_0201_0603Metric_L, F.Cu at (138.5, 93.6)
- added R8: 200kR, amemb-Resistor_SMD:amemb-R_0201_0603Metric_L, F.Cu at (138.8, 93.9)
- added R9: 100kR, amemb-Resistor_SMD:amemb-R_0201_0603Metric_L, F.Cu at (138.1, 99.9)
- U2: moved to F.Cu
- U3: moved to B.Cu
- moved LOGO1 38.7 mm to (141.4, 108.0), turned to 0 degrees
- moved H2 24.8 mm to (118.1, 77.7)
- moved AE1 12.6 mm to (160.2, 117.5), turned to 90 degrees
- moved U3 9.96 mm to (148.5, 98.7), turned to 90 degrees
- moved U10 8.86 mm to (143.5, 111.3)
- moved D1 7.80 mm to (152.3, 94.6)
- moved U5 6.19 mm to (152.4, 111.2), turned to 90 degrees
- moved U6 5.02 mm to (153.5, 104.5)
- moved U9 3.48 mm to (139.2, 105.2), turned to -90 degrees
- moved U7 2.91 mm to (154.3, 116.5)
- moved U8 2.03 mm to (141.4, 96.5), turned to 135 degrees
- moved J2 1.40 mm to (148.5, 94.6), turned to 0 degrees
- moved J3 0.75 mm to (143.5, 117.8)
- moved U2 0.71 mm to (156.9, 94.1), turned to 0 degrees
Connections:
- U3 pad 1: unconnected-(U3-XO-Pad1) -> Net-(U3-XO)
- U3 pad 15: unconnected-(U3-V5-Pad15) -> Net-(U3-V5)
- U3 pad 16: unconnected-(U3-VDD33-Pad16) -> Net-(U3-VDD33)
- U3 pad 2: unconnected-(U3-XI-Pad2) -> Net-(U3-XI)
Other:
- board text added: "Framework Expansion Card Day 5 - Linux SBC"
- board text removed: "Framework Expansion Card Day 4 - Linux SBC"
