File: Day_05_Linux_SBC/Day_05_Linux_SBC.kicad_sch (KiCad schematic)
At the start: 21 parts, among them J1 USB_C_Plug_USB2.0, J2 Conn_ARM_SWD_TagConnect_TC203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, J3 USB_C_Receptacle_USB2.0_14P, J4 Conn_01x04_MountingPin, J5 Micro_SD_Card_Det2, J6 Conn_01x02_MountingPin, U1 D3V3XA4B10LP, U2 STM32H503KBUx, U3 RV1106G2, U4 CH334P

Commit message: updates
Parts:
- removed C1, C2, C4: 10uF, symbol Device:C_Small
- removed C3: 1uF, symbol Device:C_Small
- removed J2: Conn_ARM_SWD_TagConnect_TC2030-NL, Connector:Tag-Connect_TC2030-IDC-NL_2x03_P1.27mm_Vertical, symbol Connector:Conn_ARM_SWD_TagConnect_TC2030-NL
- removed J4: Conn_01x04_MountingPin, Connector_JST:JST_SH_SM04B-SRSS-TB_1x04-1MP_P1.00mm_Horizontal, symbol Connector_Generic_MountingPin:Conn_01x04_MountingPin
- removed J5: Micro_SD_Card_Det2, Connector_Card:microSD_HC_Hirose_DM3D-SF, symbol Connector:Micro_SD_Card_Det2
- removed J6: Conn_01x02_MountingPin, symbol Connector_Generic_MountingPin:Conn_01x02_MountingPin
- removed JP1: Jumper_2_Open, symbol Jumper:Jumper_2_Open
- removed R2: 10kR, symbol Device:R_Small_US
- removed U2: STM32H503KBUx, Package_DFN_QFN:QFN-32-1EP_5x5mm_P0.5mm_EP3.45x3.45mm, symbol MCU_ST_STM32H5:STM32H503KBUx
- removed U3: RV1106G2, Framework_Shilling_Library:QFN-128_L12.3-W12.3-P0.35-TL-EP7.0-1, symbol Framework_Shilling_Library:RV1106G2
- removed U4: CH334P, Package_DFN_QFN:QFN-16-1EP_3x3mm_P0.5mm_EP1.75x1.75mm, symbol Framework_Shilling_Library:CH334P
- added C25: 1uF, symbol Device:C_Small
- added C64, C65, C66: 10uF, symbol Device:C_Small
- added U10: TS3USB30ERSWR, Package_DFN_QFN:UQFN-10_1.4x1.8mm_P0.4mm, symbol Interface_USB:TS3USB30ERSWR
- added U3: CH334P, Package_DFN_QFN:QFN-16-1EP_3x3mm_P0.5mm_EP1.75x1.75mm, symbol amemb-Interface_USB:CH334P
- added U7: STEMMA-QT, amemb-Conenctor_JST:JST_SH_SM04B-SRSS-TB_1x04-1MP_P1.00mm_Horizontal, symbol amemb-Connector:STEMMA-QT
- added Y4: 12MHz, symbol Device:Crystal_GND23_Small
Connections:
- net +3V3: now also C25.1, U10.8 (~{OE}), U10.9 (VCC)
- net D+: now also U3.12 (DPU+)
- net D-: now also U3.11 (DMU-)
- net GND: now also C25.2, C64.2, C65.2, C66.2, U10.4 (GND), U3.17 (GND), Y4.2 (G), Y4.3 (G)
- net PMIC.CC1: now reaches J3.A5 (CC1)
- net MPU_OUT.D+: now reaches J3.A6 (D+)
- net MPU_OUT.D+: now also J3.B6 (D+), U10.1 (D1+)
- net MPU_OUT.D-: now reaches J3.A7 (D-)
- net MPU_OUT.D-: now also J3.B7 (D-), U10.7 (D1-)
- net PMIC.CC2: now reaches J3.B5 (CC2)
- new net: C64.1, U3.15 (V5)
- new net: C65.1, C66.1, U3.16 (VDD33)
- new net: U10.2 (D2+), U3.10 (DP1+)
- new net: U10.6 (D2-), U3.9 (DM1-)
- new net: U7.1 (GND), U7.5 (GND)
- new net: U3.1 (XO), Y4.1
- new net: U3.2 (XI), Y4.4
- new net DEBUG.D+: U3.8 (DP2+)
- new net DEBUG.D-: U3.7 (DM2-)
- new net ESP32.D+: U3.6 (DP3+)
- new net ESP32.D-: U3.5 (DM3-)
- new net MPU.D+: U10.3 (D+)
- new net MPU.D-: U10.5 (D-)
- new net MPU_USB_SW: U10.10 (S)
- no-connect marks 4 -> 5
Other:
- added sheet ESP32-C6 (sch/WiFi_ESP32-C6.kicad_sch)
- added sheet Power Supply (sch/Power_Supply.kicad_sch)
- added sheet RV1106G2 (sch/MPU_RV1106G2.kicad_sch)
- added sheet STM32H5 (sch/MCU_STM32H5.kicad_sch)
- note removed: "battery"
- moved on the sheet: J3, U1

Commit message: updates
Parts:
- C25: footprint (none) -> amemb-Capacitor_SMD:amemb-C_0201_0603Metric_L; LCSC (none) -> C6119758
- C64, C65, C66: footprint (none) -> amemb-Capacitor_SMD:amemb-C_0402_1005Metric_L; LCSC (none) -> C315248
- R1: footprint (none) -> amemb-Resistor_SMD:amemb-R_0201_0603Metric_L; LCSC (none) -> C5356117
Changed lines of the file:
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@@
 			)
 		)
-		(property "Footprint" ""
+		(property "Footprint" "amemb-Capacitor_SMD:amemb-C_0402_1005Metric_L"
 			(at 135.89 27.94 0)
 			(hide yes)
@@
 		)
 		(property "Description" "Unpolarized capacitor, small symbol"
+			(at 135.89 27.94 0)
+			(hide yes)
+			(show_name no)
+			(do_not_autoplace no)
+			(effects
+				(font
+					(size 1.27 1.27)
+				)
+			)
+		)
+		(property "LCSC" "C315248"
 			(at 135.89 27.94 0)
 			(hide yes)
@@
 			)
 		)
-		(property "Footprint" ""
+		(property "Footprint" "amemb-Capacitor_SMD:amemb-C_0402_1005Metric_L"
 			(at 120.65 27.94 0)
 			(hide yes)
@@
 		)
 		(property "Description" "Unpolarized capacitor, small symbol"
+			(at 120.65 27.94 0)
+			(hide yes)
+			(show_name no)
+			(do_not_autoplace no)
+			(effects
+				(font
+					(size 1.27 1.27)
+				)
+			)
+		)
+		(property "LCSC" "C315248"
 			(at 120.65 27.94 0)
 			(hide yes)
@@
 			)
 		)
-		(property "Footprint" ""
+		(property "Footprint" "amemb-Resistor_SMD:amemb-R_0201_0603Metric_L"
 			(at 57.15 52.07 0)
 			(hide yes)
@@
 		)
 		(property "Description" "Resistor, small US symbol"
+			(at 57.15 52.07 0)
+			(hide yes)
+			(show_name no)
+			(do_not_autoplace no)
+			(effects
+				(font
+					(size 1.27 1.27)
+				)
+			)
+		)
+		(property "LCSC" "C5356117"
 			(at 57.15 52.07 0)
 			(hide yes)
@@
 			)
 		)
-		(property "Footprint" ""
+		(property "Footprint" "amemb-Capacitor_SMD:amemb-C_0201_0603Metric_L"
 			(at 160.02 30.48 0)
 			(hide yes)
@@
 		)
 		(property "Description" "Unpolarized capacitor, small symbol"
+			(at 160.02 30.48 0)
+			(hide yes)
+			(show_name no)
+			(do_not_autoplace no)
+			(effects
+				(font
+					(size 1.27 1.27)
+				)
+			)
+		)
+		(property "LCSC" "C6119758"
 			(at 160.02 30.48 0)
 			(hide yes)
@@
 			)
 		)
-		(property "Footprint" ""
+		(property "Footprint" "amemb-Capacitor_SMD:amemb-C_0402_1005Metric_L"
 			(at 110.49 27.94 0)
 			(hide yes)
@@
 			(at 110.49 27.94 0)
 			(hide yes)
+			(show_name no)
+			(do_not_autoplace no)
+			(effects
+				(font
+					(size 1.27 1.27)
+				)
+			)
+		)
+		(property "LCSC" "C315248"
+			(at 110.49 27.94 0)
+			(hide yes)
