File: Day_05_Linux_SBC/sch/MCU_STM32H5.kicad_sch (KiCad schematic)
At the start: 8 parts, among them J2 Conn_ARM_SWD_TagConnect_TC203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, U2 STM32H503KBUx

Commit message: updates
Parts:
- C1, C2, C4: footprint (none) -> amemb-Capacitor_SMD:amemb-C_0402_1005Metric_L; LCSC (none) -> C315248
- C3: footprint (none) -> amemb-Capacitor_SMD:amemb-C_0201_0603Metric_L; LCSC (none) -> C6119758
- R2: footprint (none) -> amemb-Resistor_SMD:amemb-R_0201_0603Metric_L; LCSC (none) -> C49653507
