File: Day_05_Linux_SBC/sch/MPU_RV1106G2.kicad_sch (KiCad schematic)
At the start: 31 parts, among them J5 Micro_SD_Card_Det2, U6 RV1106G2, Y1 24MHz, Y2 32.768kHz

Commit message: updates
Parts:
- C38, C44, C45, C49, C55, C57: footprint (none) -> amemb-Capacitor_SMD:amemb-C_0402_1005Metric_L; LCSC (none) -> C315248
- C39, C40, C41, C42, C43, C46, C47, C48, C50, C51, C52, C53, C54, C56, C58, C59, C60, C61, C62, C63: footprint (none) -> amemb-Capacitor_SMD:amemb-C_0201_0603Metric_L; LCSC (none) -> C6119758
- R14: footprint (none) -> amemb-Resistor_SMD:amemb-R_0201_0603Metric_L; LCSC (none) -> C7467273
