File: Day_05_Linux_SBC/sch/Power_Supply.kicad_sch (KiCad schematic)
At the start: 39 parts, among them J4 JST SH SM03B, U8 EA3058QD, U9 MP2722

Commit message: updates
Parts:
- C10, C5, C6, C7: footprint (none) -> amemb-Capacitor_SMD:amemb-C_0201_0603Metric_L; LCSC (none) -> C20616244
- C11, C12, C13, C14, C22: footprint (none) -> amemb-Capacitor_SMD:amemb-C_0402_1005Metric_L; LCSC (none) -> C3845593
- C15, C16, C17, C18, C19, C23: footprint (none) -> amemb-Capacitor_SMD:amemb-C_0402_1005Metric_L; LCSC (none) -> C315248
- C20: footprint (none) -> amemb-Capacitor_SMD:amemb-C_0201_0603Metric_L; LCSC (none) -> C2880350
- C21: footprint (none) -> amemb-Capacitor_SMD:amemb-C_0201_0603Metric_L; LCSC (none) -> C6119758
- C24: footprint (none) -> amemb-Capacitor_SMD:amemb-C_0402_1005Metric_L; LCSC (none) -> C6119786
- C8: footprint (none) -> amemb-Capacitor_SMD:amemb-C_0201_0603Metric_L; LCSC (none) -> C5142564
- C9: footprint (none) -> amemb-Capacitor_SMD:amemb-C_0201_0603Metric_L; LCSC (none) -> C18164587
- L1, L2, L3, L4: footprint (none) -> amemb-Inductor_SMD:amemb-L_0806_2016Metric_L; LCSC (none) -> C48945509
- L5: footprint (none) -> amemb-Inductor_SMD:amemb-L_0805_2012Metric_L; LCSC (none) -> C5441853
- R10, R12, R4, R5, R7, R9: footprint (none) -> amemb-Resistor_SMD:amemb-R_0201_0603Metric_L; LCSC (none) -> C3152012
- R11, R8: footprint (none) -> amemb-Resistor_SMD:amemb-R_0201_0603Metric_L; LCSC (none) -> C3152021
- R13, R3: footprint (none) -> amemb-Resistor_SMD:amemb-R_0201_0603Metric_L; LCSC (none) -> C7421800
- R6: value 80kR -> 80.6kR; footprint (none) -> amemb-Resistor_SMD:amemb-R_0201_0603Metric_L; LCSC (none) -> C19626324
