File: Day_05_Linux_SBC/sch/WiFi_ESP32-C6.kicad_sch (KiCad schematic)
At the start: 19 parts, among them U5 ESP32-C6FH4, Y3 40MHZ

Commit message: updates
Parts:
- C26: footprint (none) -> amemb-Capacitor_SMD:amemb-C_0402_1005Metric_L; LCSC (none) -> C315248
- C27, C28, C29, C30, C31, C32, C33: footprint (none) -> amemb-Capacitor_SMD:amemb-C_0201_0603Metric_L; LCSC (none) -> C6119758
- C34, C35, C36, C37: footprint (none) -> amemb-Capacitor_SMD:amemb-C_01005_0402Metric_L; LCSC (none) -> C1517597
- L6: footprint (none) -> amemb-Inductor_SMD:amemb-L_0201_0603Metric_L; LCSC (none) -> C279889
- L7: footprint (none) -> amemb-Resistor_SMD:amemb-R_0201_0603Metric_L; LCSC (none) -> C3152011
- R15, R16: footprint (none) -> amemb-Resistor_SMD:amemb-R_0201_0603Metric_L; LCSC (none) -> C3152012
Changed lines of the file:
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@@
 	)
 	(junction
-		(at 44.45 81.28)
-		(diameter 0)
-		(color 0 0 0 0)
-	)
-	(junction
 		(at 68.58 81.28)
 		(diameter 0)
@@
 	)
 	(no_connect
-		(at 35.56 81.28)
+		(at 39.37 81.28)
 	)
 	(no_connect
@@
 	(wire
 		(pts
-			(xy 35.56 81.28) (xy 39.37 81.28)
-		)
-		(stroke
-			(width 0)
-			(type default)
-		)
-	)
-	(wire
-		(pts
 			(xy 175.26 60.96) (xy 175.26 76.2)
 		)
@@
 	(wire
 		(pts
-			(xy 40.64 81.28) (xy 44.45 81.28)
-		)
-		(stroke
-			(width 0)
-			(type default)
-		)
-	)
-	(wire
-		(pts
 			(xy 143.51 60.96) (xy 152.4 60.96)
 		)
@@
 			)
 		)
-		(property "Footprint" ""
+		(property "Footprint" "amemb-Capacitor_SMD:amemb-C_0201_0603Metric_L"
 			(at 143.51 63.5 0)
 			(hide yes)
@@
 			)
 		)
+		(property "LCSC" "C6119758"
+			(at 143.51 63.5 0)
+			(hide yes)
+			(show_name no)
+			(do_not_autoplace no)
+			(effects
+				(font
+					(size 1.27 1.27)
+				)
+			)
+		)
 		(pin "1"
 		)
@@
 			)
 		)
-		(property "Footprint" ""
+		(property "Footprint" "amemb-Capacitor_SMD:amemb-C_01005_0402Metric_L"
 			(at 101.6 83.82 0)
 			(hide yes)
@@
 			)
 		)
+		(property "LCSC" "C1517597"
+			(at 101.6 83.82 0)
+			(hide yes)
+			(show_name no)
+			(do_not_autoplace no)
+			(effects
+				(font
+					(size 1.27 1.27)
+				)
+			)
+		)
 		(pin "1"
 		)
@@
 			)
 		)
-		(property "Footprint" ""
+		(property "Footprint" "amemb-Capacitor_SMD:amemb-C_0402_1005Metric_L"
 			(at 107.95 63.5 0)
 			(hide yes)
@@
 			)
 		)
+		(property "LCSC" "C315248"
+			(at 107.95 63.5 0)
+			(hide yes)
+			(show_name no)
+			(do_not_autoplace no)
+			(effects
+				(font
+					(size 1.27 1.27)
+				)
+			)
+		)
 		(pin "1"
 		)
@@
 			)
 		)
-		(property "Footprint" ""
+		(property "Footprint" "amemb-Resistor_SMD:amemb-R_0201_0603Metric_L"
 			(at 59.69 81.28 0)
 			(hide yes)
@@
 			)
 		)
+		(property "LCSC" "C3152011"
+			(at 59.69 81.28 0)
+			(hide yes)
+			(show_name no)
+			(do_not_autoplace no)
+			(effects
+				(font
+					(size 1.27 1.27)
+				)
+			)
+		)
 		(pin "2"
 		)
@@
 			)
 		)
-		(property "Footprint" ""
+		(property "Footprint" "amemb-Inductor_SMD:amemb-L_0201_0603Metric_L"
 			(at 92.71 81.28 0)
 			(hide yes)
@@
 			)
 		)
+		(property "LCSC" "C279889"
+			(at 92.71 81.28 0)
+			(hide yes)
+			(show_name no)
+			(do_not_autoplace no)
+			(effects
+				(font
+					(size 1.27 1.27)
+				)
+			)
+		)
 		(pin "2"
 		)
@@
 			)
 		)
-		(property "Footprint" ""
+		(property "Footprint" "amemb-Capacitor_SMD:amemb-C_0201_0603Metric_L"
 			(at 116.84 63.5 0)
 			(hide yes)
@@
 			)
 		)
+		(property "LCSC" "C6119758"
+			(at 116.84 63.5 0)
+			(hide yes)
+			(show_name no)
+			(do_not_autoplace no)
+			(effects
+				(font
+					(size 1.27 1.27)
+				)
+			)
+		)
 		(pin "1"
 		)
@@
 			)
 		)
-		(property "Footprint" ""
+		(property "Footprint" "amemb-Capacitor_SMD:amemb-C_01005_0402Metric_L"
 			(at 68.58 83.82 0)
 			(hide yes)
@@
 			)
 		)
+		(property "LCSC" "C1517597"
+			(at 68.58 83.82 0)
+			(hide yes)
+			(show_name no)
+			(do_not_autoplace no)
+			(effects
+				(font
+					(size 1.27 1.27)
+				)
+			)
+		)
 		(pin "1"
 		)
@@
 			)
 		)
-		(property "Footprint" ""
+		(property "Footprint" "amemb-Capacitor_SMD:amemb-C_01005_0402Metric_L"
 			(at 83.82 83.82 0)
 			(hide yes)
@@
 			)
 		)
+		(property "LCSC" "C1517597"
+			(at 83.82 83.82 0)
+			(hide yes)
+			(show_name no)
+			(do_not_autoplace no)
+			(effects
+				(font
+					(size 1.27 1.27)
+				)
+			)
+		)
 		(pin "1"
 		)
@@
 			)
 		)
-		(property "Footprint" ""
+		(property "Footprint" "amemb-Resistor_SMD:amemb-R_0201_0603Metric_L"
 			(at 214.63 109.22 0)
 			(hide yes)
@@
 			)
 		)
+		(property "LCSC" "C3152012"
+			(at 214.63 109.22 0)
+			(hide yes)
+			(show_name no)
+			(do_not_autoplace no)
+			(effects
+				(font
+					(size 1.27 1.27)
+				)
+			)
+		)
 		(pin "1"
 		)
@@
 			)
 		)
-		(property "Footprint" ""
+		(property "Footprint" "amemb-Capacitor_SMD:amemb-C_0201_0603Metric_L"
 			(at 125.73 63.5 0)
 			(hide yes)
@@
 			)
 		)
+		(property "LCSC" "C6119758"
+			(at 125.73 63.5 0)
+			(hide yes)
+			(show_name no)
+			(do_not_autoplace no)
+			(effects
+				(font
+					(size 1.27 1.27)
+				)
+			)
+		)
 		(pin "1"
 		)
@@
 			)
 		)
-		(property "Footprint" ""
+		(property "Footprint" "amemb-Capacitor_SMD:amemb-C_0201_0603Metric_L"
 			(at 161.29 63.5 0)
 			(hide yes)
@@
 			)
 		)
+		(property "LCSC" "C6119758"
+			(at 161.29 63.5 0)
+			(hide yes)
+			(show_name no)
+			(do_not_autoplace no)
+			(effects
+				(font
+					(size 1.27 1.27)
+				)
+			)
+		)
 		(pin "1"
 		)
@@
 			)
 		)
-		(property "Footprint" ""
+		(property "Footprint" "amemb-Resistor_SMD:amemb-R_0201_0603Metric_L"
 			(at 116.84 91.44 0)
 			(hide yes)
@@
 			)
 		)
+		(property "LCSC" "C3152012"
+			(at 116.84 91.44 0)
+			(hide yes)
+			(show_name no)
+			(do_not_autoplace no)
+			(effects
+				(font
+					(size 1.27 1.27)
+				)
+			)
+		)
 		(pin "1"
 		)
@@
 			)
 		)
-		(property "Footprint" ""
+		(property "Footprint" "amemb-Capacitor_SMD:amemb-C_0201_0603Metric_L"
 			(at 152.4 63.5 0)
 			(hide yes)
@@
 			)
 		)
+		(property "LCSC" "C6119758"
+			(at 152.4 63.5 0)
+			(hide yes)
+			(show_name no)
+			(do_not_autoplace no)
+			(effects
+				(font
+					(size 1.27 1.27)
+				)
+			)
+		)
 		(pin "1"
 		)
@@
 			)
 		)
-		(property "Footprint" ""
+		(property "Footprint" "amemb-Capacitor_SMD:amemb-C_01005_0402Metric_L"
 			(at 50.8 83.82 0)
 			(hide yes)
@@
 			)
 		)
+		(property "LCSC" "C1517597"
+			(at 50.8 83.82 0)
+			(hide yes)
+			(show_name no)
+			(do_not_autoplace no)
+			(effects
+				(font
+					(size 1.27 1.27)
+				)
+			)
+		)
 		(pin "1"
 		)
@@
 			)
 		)
-		(property "Footprint" ""
+		(property "Footprint" "amemb-Capacitor_SMD:amemb-C_0201_0603Metric_L"
 			(at 134.62 63.5 0)
 			(hide yes)
@@
 			)
 		)
+		(property "LCSC" "C6119758"
+			(at 134.62 63.5 0)
+			(hide yes)
+			(show_name no)
+			(do_not_autoplace no)
+			(effects
+				(font
+					(size 1.27 1.27)
+				)
+			)
+		)
 		(pin "1"
 		)
@@
 			)
 		)
-		(property "Footprint" ""
+		(property "Footprint" "amemb-Capacitor_SMD:amemb-C_0201_0603Metric_L"
 			(at 170.18 63.5 0)
 			(hide yes)
@@
 			(at 170.18 63.5 0)
 			(hide yes)
+			(show_name no)
+			(do_not_autoplace no)
+			(effects
+				(font
+					(size 1.27 1.27)
+				)
+			)
+		)
+		(property "LCSC" "C6119758"
+			(at 170.18 63.5 0)
+			(hide yes)
